File: Sira_7K_Pad.kicad_sch (KiCad schematic)
At the start: 0 parts

Commit message: added usb c libraries
Parts:
- added C1: 1uF, symbol Device:C_Small
- added C2, C3: 22pF, symbol Device:C_Small
- added C4, C5, C6, C7: 0.1uF, symbol Device:C_Small
- added C8: 10uF, symbol Device:C_Small
- added J1: AVR-ISP-6, symbol Connector:AVR-ISP-6
- added R1, R4: 10k, symbol Device:R_Small
- added R2, R3: 22, symbol Device:R_Small
- added SW1: SW_Push, symbol Switch:SW_Push
- added U1: ATmega32U4-A, Package_QFP:TQFP-44_10x10mm_P0.8mm, symbol MCU_Microchip_ATmega:ATmega32U4-A
- added Y1: Crystal_GND24_Small, symbol Device:Crystal_GND24_Small
Connections:
- new net: R2.2, U1.4 (D+)
- new net: R3.2, U1.3 (D-)
- new net: R1.1, U1.33 (~{HWB}/PE2)
- new net: C1.1, U1.6 (UCAP)
- new net +5V: C4.1, C5.1, C6.1, C7.1, C8.1, J1.2 (VCC), U1.14 (VCC), U1.2 (UVCC), U1.24 (AVCC), U1.34 (VCC), U1.44 (AVCC), U1.7 (VBUS)
- new net GND: C1.2, C2.2, C3.2, C4.2, C5.2, C6.2, C7.2, C8.2, J1.6 (GND), R1.2, SW1.1, U1.15 (GND), U1.23 (GND), U1.35 (GND), U1.43 (GND), U1.5 (UGND), Y1.2, Y1.4
- new net MISO: J1.1 (MISO), U1.9 (PB1)
- new net MOSI: J1.4 (MOSI), U1.10 (PB2)
- new net RESET: J1.5 (~{RST}), R4.2, SW1.2, U1.13 (~{RESET})
- new net SCK: J1.3 (SCK), U1.11 (PB3)
- new net XTAL1: C2.1, U1.17 (XTAL1), Y1.1
- new net XTAL2: C3.1, U1.16 (XTAL2), Y1.3
- no-connect marks 0 -> 1

Commit message: finished schematic
Parts:
- added F1: 500mA, symbol Device:Polyfuse_Small
- added R5, R6: 5.1k, symbol Device:R_Small
- added U2: PRTR5V0U2X, symbol random-keyboard-parts:PRTR5V0U2X
- added USB1: HRO-TYPE-C-31-M-12, symbol Type-C:HRO-TYPE-C-31-M-12
Connections:
- net +5V: now also R4.1, F1.2
- net GND: now also R5.2, R6.2, U2.1 (GND), USB1.1 (GND), USB1.12 (GND), USB1.13 (SHIELD)
- net MISO: now also U1.11 (PB3); no longer U1.9 (PB1)
- net SCK: now also U1.9 (PB1); no longer U1.11 (PB3)
- net D+: now reaches R2.1
- net D+: now also U2.2 (IO1), USB1.6 (DP1), USB1.8 (DP2)
- net D-: now reaches R3.1
- net D-: now also U2.3 (IO2), USB1.5 (DN2), USB1.7 (DN1)
- new net: R6.1, USB1.4 (CC1)
- new net: R5.1, USB1.10 (CC2)
- new net VCC: F1.1, U2.4 (VCC), USB1.11 (VBUS), USB1.2 (VBUS)
- no-connect marks 1 -> 3
Other:
- moved on the sheet: R4
