File: Sira_7K_Pad.kicad_pcb (KiCad board)
At the start: 2 copper layers, 136.5 x 85.7 mm, 29 parts, among them J1 AVR-ISP-6, SW1 SW_Push, U1 ATmega32U4-A, U2 PRTR5V0U2X, Y1 Crystal_GND24_Small

Commit message: finished (first version) pbc
Parts:
- added FB1: 60@100MHz, Inductor_SMD:L_0805_2012Metric, F.Cu at (159.5, 65.4)
- moved R4 0.46 mm to (130.5, 84.2)
Connections:
- USB1 pad 13: GND -> Earth
Routing:
- net GND: track 368.2 -> 363.5 mm, vias 9 -> 42
- net +5V: track 151.1 -> 152.2 mm
- net Earth: vias 0 -> 5
- added copper zone on F.Cu, net Earth
