File: Sira_7K_Pad.kicad_pcb (KiCad board)
At the start: 2 copper layers, 136.5 x 87.3 mm, 30 parts, among them J1 AVR-ISP-6, SW1 SW_Push, U1 ATmega32U4-A, U2 PRTR5V0U2X, Y1 Crystal_GND24_Small

Commit message: idk
Connections:
- USB1 pad 13: Earth -> GND
Changed lines of the file:
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@@
 			(layers "*.Cu" "*.Mask")
 			(remove_unused_layers no)
-			(net 43 "Earth")
+			(net 2 "GND")
 			(pinfunction "SHIELD")
 			(pintype "input")
@@
 			(layers "*.Cu" "*.Mask")
 			(remove_unused_layers no)
-			(net 43 "Earth")
+			(net 2 "GND")
 			(pinfunction "SHIELD")
 			(pintype "input")
@@
 			(layers "*.Cu" "*.Mask")
 			(remove_unused_layers no)
-			(net 43 "Earth")
+			(net 2 "GND")
 			(pinfunction "SHIELD")
 			(pintype "input")
@@
 			(layers "*.Cu" "*.Mask")
 			(remove_unused_layers no)
-			(net 43 "Earth")
+			(net 2 "GND")
 			(pinfunction "SHIELD")
 			(pintype "input")
